Commit message: Model the wheels as wheels, one link each
The four corners were mock geometry baked into base_link: vertical
cylinders, r=155 mm, h=254 mm, which read as housings rather than
anything that could roll. They are wheels, 250 mm in diameter and 200 mm
wide, so they are now cylinders of r=125 mm and length 200 mm rolled 90
degrees about X to lay the axle across the rover.

Each is its own link. That is needed twice over: a wheel inside base_link
cannot carry a steering or rolling joint, and a URDF link applies its
first visual's material to every visual it holds, so geometry sharing
base_link could not be coloured separately either - which is why an
attempt to highlight them came out blue.

The axle stays at the mock's z = -0.284, putting the contact patch at
-0.409, within 2 mm of where the mock sat, so no ride height is invented.
base_footprint_joint moves from 0 to 0.409 so base_footprint lies on the
ground plane as its name promises; at zero the rover would spawn 409 mm
into the floor of any world.

The joints are fixed for now. Steering and rolling come with the
simulation that will drive them.

File: asterope_iiI.urdf (robot description, URDF)
Before this commit: robot asterope, 14 links, 13 joints
Links:
- added link wheel_front_left; collision cylinder length=0.200 radius=0.125; visual cylinder length=0.200 radius=0.125
- added link wheel_front_right; collision cylinder length=0.200 radius=0.125; visual cylinder length=0.200 radius=0.125
- added link wheel_rear_left; collision cylinder length=0.200 radius=0.125; visual cylinder length=0.200 radius=0.125
- added link wheel_rear_right; collision cylinder length=0.200 radius=0.125; visual cylinder length=0.200 radius=0.125
- link base_link: geometry collision box size=0.037 0.188 0.03; collision box size=0.037 0.188 0.03
Joints:
- added joint wheel_front_left_joint: type fixed, parent base_link, child wheel_front_left, origin xyz=0.455 0.455 -0.284 rpy=0 0 0
- added joint wheel_front_right_joint: type fixed, parent base_link, child wheel_front_right, origin xyz=0.455 -0.455 -0.284 rpy=0 0 0
- added joint wheel_rear_left_joint: type fixed, parent base_link, child wheel_rear_left, origin xyz=-0.455 0.455 -0.284 rpy=0 0 0
- added joint wheel_rear_right_joint: type fixed, parent base_link, child wheel_rear_right, origin xyz=-0.455 -0.455 -0.284 rpy=0 0 0
- joint base_footprint_joint: origin xyz=0 0 0.0 rpy=0 0 0 -> xyz=0 0 0.409 rpy=0 0 0

Commit message: Give each wheel a steering joint and a rolling joint
The four wheels were on fixed joints, so nothing could steer or roll.
Each corner is now a steering link revolute about Z carrying a wheel
continuous about Y. Steering is limited to one turn either way because
the steer module is cabled rather than on a slip ring.

Tested by parsing the URDF rather than through ROS, so the checks run in
the ground station's venv, which has no ROS by design.

File: asterope_iiI.urdf (robot description, URDF)
Before this commit: robot asterope, 18 links, 17 joints
Links:
- added link steer_front_left; visual cylinder length=0.16 radius=0.06
- added link steer_front_right; visual cylinder length=0.16 radius=0.06
- added link steer_rear_left; visual cylinder length=0.16 radius=0.06
- added link steer_rear_right; visual cylinder length=0.16 radius=0.06
Joints:
- added joint steer_front_left_joint: type revolute, parent base_link, child steer_front_left, origin xyz=0.455 0.455 -0.284 rpy=0 0 0, axis 0 0 1, limit lower=-3.14159265 upper=3.14159265 effort=100 velocity=6.0
- added joint steer_front_right_joint: type revolute, parent base_link, child steer_front_right, origin xyz=0.455 -0.455 -0.284 rpy=0 0 0, axis 0 0 1, limit lower=-3.14159265 upper=3.14159265 effort=100 velocity=6.0
- added joint steer_rear_left_joint: type revolute, parent base_link, child steer_rear_left, origin xyz=-0.455 0.455 -0.284 rpy=0 0 0, axis 0 0 1, limit lower=-3.14159265 upper=3.14159265 effort=100 velocity=6.0
- added joint steer_rear_right_joint: type revolute, parent base_link, child steer_rear_right, origin xyz=-0.455 -0.455 -0.284 rpy=0 0 0, axis 0 0 1, limit lower=-3.14159265 upper=3.14159265 effort=100 velocity=6.0
- joint wheel_front_left_joint: axis (none) -> 0 1 0; origin xyz=0.455 0.455 -0.284 rpy=0 0 0 -> xyz=0 0 0 rpy=0 0 0; parent base_link -> steer_front_left; type fixed -> continuous
- joint wheel_front_right_joint: axis (none) -> 0 1 0; origin xyz=0.455 -0.455 -0.284 rpy=0 0 0 -> xyz=0 0 0 rpy=0 0 0; parent base_link -> steer_front_right; type fixed -> continuous
- joint wheel_rear_left_joint: axis (none) -> 0 1 0; origin xyz=-0.455 0.455 -0.284 rpy=0 0 0 -> xyz=0 0 0 rpy=0 0 0; parent base_link -> steer_rear_left; type fixed -> continuous
- joint wheel_rear_right_joint: axis (none) -> 0 1 0; origin xyz=-0.455 -0.455 -0.284 rpy=0 0 0 -> xyz=0 0 0 rpy=0 0 0; parent base_link -> steer_rear_right; type fixed -> continuous

Commit message: Fix round 1: make the wheels survive into Gazebo and let their joints move
Three defects, all found by running the simulation rather than by reading it.

Gazebo's URDF-to-SDF conversion silently drops any link on a non-fixed
joint that carries no <inertial> - no error, no warning, the link simply
vanishes. All eight steer and wheel links lacked one, so the rover
spawned as a single body with no wheels at all. They now carry nominal
inertials, commented as such: they exist so the links survive conversion
and are not hardware measurements. A URDF test asserts positive mass on
each, because a failure this quiet needs a guard that is not somebody
looking at Gazebo. This is not the contact-physics tuning the design
rules out - it is the structural minimum a link needs to exist.

gazebo_ros_joint_pose_trajectory rejects any trajectory without a
reference link, so every message was refused and no joint moved. The
reference is base_footprint rather than the more natural base_link:
base_footprint_joint is fixed, so the conversion lumps base_link's
geometry into base_footprint and no base_link survives to be named.

The same plugin compares each trajectory's stamp against the simulation
clock, so without use_sim_time the node's wall-clock stamps landed far
in the sim's future and nothing was ever applied.

The topic the simulation drives from is now a launch argument defaulting
to the rover's own /manual_twist. A hardcoded scratch topic had been
left in place from testing, which would have shipped a simulation that
never heard the rover; the argument keeps the safe path available
without making it the default.

File: asterope_iiI.urdf (robot description, URDF)
Before this commit: robot asterope, 22 links, 21 joints
Links:
- link steer_front_left: mass None -> 1.0
- link steer_front_right: mass None -> 1.0
- link steer_rear_left: mass None -> 1.0
- link steer_rear_right: mass None -> 1.0
- link wheel_front_left: mass None -> 4.0
- link wheel_front_right: mass None -> 4.0
- link wheel_rear_left: mass None -> 4.0
- link wheel_rear_right: mass None -> 4.0

Commit message: Add the two ZED 2i camera frames to the URDF, front offset flagged as unverified

File: asterope_iiI.urdf (robot description, URDF)
Before this commit: robot asterope, 22 links, 21 joints
Links:
- removed link zed_front_camera_center
- removed link zed_front_camera_link
- removed link zed_front_left_camera_frame
- removed link zed_front_left_camera_frame_optical
- removed link zed_front_right_camera_frame
- removed link zed_front_right_camera_frame_optical
- removed link zed_rear_camera_center
- removed link zed_rear_left_camera_frame
- removed link zed_rear_left_camera_frame_optical
- removed link zed_rear_right_camera_frame
- removed link zed_rear_right_camera_frame_optical
- added link zed_camera_link
Joints:
- removed joint zed_front_camera_center_joint
- removed joint zed_front_camera_joint
- removed joint zed_front_left_camera_joint
- removed joint zed_front_left_camera_optical_joint
- removed joint zed_front_right_camera_joint
- removed joint zed_front_right_camera_optical_joint
- removed joint zed_rear_camera_center_joint
- removed joint zed_rear_left_camera_joint
- removed joint zed_rear_left_camera_optical_joint
- removed joint zed_rear_right_camera_joint
- removed joint zed_rear_right_camera_optical_joint
- added joint zed_camera_joint: type fixed, parent base_link, child zed_camera_link, origin xyz=0.322 0 0.154 rpy=0 0 0
- joint zed_rear_camera_joint: origin xyz=-0.345 0 0.139 rpy=0 0 3.141592654 -> xyz=-0.322 0 0.154 rpy=0 0 3.14159265

Commit message: Restore the hardware team's measured ZED frame tree in the URDF

File: asterope_iiI.urdf (robot description, URDF)
Before this commit: robot asterope, 12 links, 11 joints
Links:
- removed link zed_camera_link
- added link zed_front_camera_center
- added link zed_front_camera_link
- added link zed_front_left_camera_frame
- added link zed_front_left_camera_frame_optical
- added link zed_front_right_camera_frame
- added link zed_front_right_camera_frame_optical
- added link zed_rear_camera_center
- added link zed_rear_left_camera_frame
- added link zed_rear_left_camera_frame_optical
- added link zed_rear_right_camera_frame
- added link zed_rear_right_camera_frame_optical
Joints:
- removed joint zed_camera_joint
- added joint zed_front_camera_center_joint: type fixed, parent zed_front_camera_link, child zed_front_camera_center, origin xyz=0 0 0.015 rpy=0 0 0
- added joint zed_front_camera_joint: type fixed, parent base_link, child zed_front_camera_link, origin xyz=0.345 0 0.139 rpy=0 0 0
- added joint zed_front_left_camera_joint: type fixed, parent zed_front_camera_center, child zed_front_left_camera_frame, origin xyz=-0.01 0.06 0 rpy=0 0 0
- added joint zed_front_left_camera_optical_joint: type fixed, parent zed_front_left_camera_frame, child zed_front_left_camera_frame_optical, origin xyz=0 0 0 rpy=-1.570796327 0 -1.570796327
- added joint zed_front_right_camera_joint: type fixed, parent zed_front_camera_center, child zed_front_right_camera_frame, origin xyz=-0.01 -0.06 0 rpy=0 0 0
- added joint zed_front_right_camera_optical_joint: type fixed, parent zed_front_right_camera_frame, child zed_front_right_camera_frame_optical, origin xyz=0 0 0 rpy=-1.570796327 0 -1.570796327
- added joint zed_rear_camera_center_joint: type fixed, parent zed_rear_camera_link, child zed_rear_camera_center, origin xyz=0 0 0.015 rpy=0 0 0
- added joint zed_rear_left_camera_joint: type fixed, parent zed_rear_camera_center, child zed_rear_left_camera_frame, origin xyz=-0.01 0.06 0 rpy=0 0 0
- added joint zed_rear_left_camera_optical_joint: type fixed, parent zed_rear_left_camera_frame, child zed_rear_left_camera_frame_optical, origin xyz=0 0 0 rpy=-1.570796327 0 -1.570796327
- added joint zed_rear_right_camera_joint: type fixed, parent zed_rear_camera_center, child zed_rear_right_camera_frame, origin xyz=-0.01 -0.06 0 rpy=0 0 0
- added joint zed_rear_right_camera_optical_joint: type fixed, parent zed_rear_right_camera_frame, child zed_rear_right_camera_frame_optical, origin xyz=0 0 0 rpy=-1.570796327 0 -1.570796327
- joint zed_rear_camera_joint: origin xyz=-0.322 0 0.154 rpy=0 0 3.14159265 -> xyz=-0.345 0 0.139 rpy=0 0 3.141592654
