Commit message: Draw the mapped terrain orange-brown and the rover black so both stand out from Gazebo's grey background
Co-Authored-By: Claude Fable 5 <noreply@anthropic.com>
Claude-Session: https://claude.ai/code/session_0116NeKBvg6uGb53WFLdcRis

File: sim/src/navi_sim_bringup/urdf/asterope_sim.urdf.xacro (robot description, xacro)
@@ -68,4 +68,15 @@
        than the real URDF because it is a statement about the simulation,
        not a fact about the rover. -->
+  <!-- The rover is drawn black in the ground station's view so it stands
+       out against the orange terrain and Gazebo's grey background. -->
+  <gazebo reference="base_link"><material>Gazebo/Black</material></gazebo>
+  <gazebo reference="steer_front_left"><material>Gazebo/Black</material></gazebo>
+  <gazebo reference="steer_front_right"><material>Gazebo/Black</material></gazebo>
+  <gazebo reference="steer_rear_left"><material>Gazebo/Black</material></gazebo>
+  <gazebo reference="steer_rear_right"><material>Gazebo/Black</material></gazebo>
+  <gazebo reference="wheel_front_left"><material>Gazebo/Black</material></gazebo>
+  <gazebo reference="wheel_front_right"><material>Gazebo/Black</material></gazebo>
+  <gazebo reference="wheel_rear_left"><material>Gazebo/Black</material></gazebo>
+  <gazebo reference="wheel_rear_right"><material>Gazebo/Black</material></gazebo>
   <gazebo reference="steer_front_left"><gravity>false</gravity></gazebo>
   <gazebo reference="wheel_front_left"><gravity>false</gravity></gazebo>
